File: PCB_Remote_Display/10MHz-Rb-Ref.sch (KiCad schematic (older format))
At the start: 29 parts, among them J1 VIN_24VDC, J2 Conn_01x06_Male, M1 Fan, SW1 SW_DPST, SW2 SW_DPST, U1 JTE0624D05, U2 INA219, U3 INA219, U4 RC1602A

Commit message: Spring Break Edition
Parts:
- removed U2, U3: INA219, Package_TO_SOT_SMD:SOT-23-8_Handsoldering, symbol 10MHz-Rb-Ref-rescue:INA219-INA219
- added J3: Conn_I2C, Connector_PinSocket_2.54mm:PinSocket_1x02_P2.54mm_Vertical, symbol Connector_Generic:Conn_01x02
- added J4: Conn_5VDC, Connector_PinSocket_2.54mm:PinSocket_1x02_P2.54mm_Vertical, symbol Connector_Generic:Conn_01x02
- added J5: Option_A, Connector_PinSocket_2.54mm:PinSocket_1x02_P2.54mm_Vertical, symbol Connector_Generic:Conn_01x02
- added J6: Option_B, Connector_PinSocket_2.54mm:PinSocket_1x02_P2.54mm_Vertical, symbol Connector_Generic:Conn_01x02
- added S1: TMP36, Package_TO_SOT_THT:TO-92_Inline, symbol MFS_Sensors:TMP36
- added TP8: TestPoint, TestPoint:TestPoint_Pad_D1.5mm, symbol Connector:TestPoint
- added U2, U3: INA219, Package_TO_SOT_SMD:SOT-23-8_Handsoldering, symbol MFS_Power:INA219
- U4: footprint Display:RC1602A -> Connector_PinSocket_2.54mm:PinSocket_2x08_P2.54mm_Vertical
Connections:
- net labels added: MICRO_D4, MICRO_D6
- wire segments 145 -> 128
- no-connect marks 0 -> 11
Other:
- note added: "Sensors and Options"
- moved on the sheet: A1, H1, H2, H3, H4, J1, J2, TP1, TP2, TP3, TP6, TP7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
